Commit message: modify rviz urdf model

File: cartographer_ros/urdf/halo_backpack_3d.urdf (robot description, URDF)
Before this commit: robot cartographer_backpack_3d, 4 links, 3 joints
Links:
- removed link vertical_vlp16_link
- link base_link: geometry visual box size=0.3 0.14 0.07
Joints:
- removed joint vertical_vlp16_link_joint
- joint horizontal_vlp16_link_joint: origin xyz=0.01 0. 0.19 rpy=0. -0.1745 3.1416 -> xyz=0.1 0. 0. rpy=0. 0. 0.
- joint imu_link_joint: origin xyz=0 0 0 rpy=3.1416 0 0 -> xyz=0 0 0 rpy=1.5758 0 0

Commit message: add emu calibration

File: cartographer_ros/urdf/halo_backpack_3d.urdf (robot description, URDF)
Before this commit: robot cartographer_backpack_3d, 3 links, 2 joints
Joints:
- joint imu_link_joint: origin xyz=0 0 0 rpy=1.5758 0 0 -> xyz=0 0 0 rpy=0 0 0
